Commit message: 第二次提交

File: catkin_ws/src/mbot_description/urdf/xacro/gazebo/mbot_base_gazebo.xacro (robot description, xacro)
@@ -1,4 +1,7 @@
 <?xml version="1.0" ?>
-<robot name="swivel" xmlns:xacro="http://www.ros.org/wiki/xacro">
+<robot name="/swivel" xmlns:xacro="http://www.ros.org/wiki/xacro"
+xmlns:sensor="http://playerstage.sourceforge.net/gazebo/xmlschema/#sensor"
+    xmlns:controller="http://playerstage.sourceforge.net/gazebo/xmlschema/#controller"
+    xmlns:interface="http://playerstage.sourceforge.net/gazebo/xmlschema/#interface">
   <!--property list -->
   <xacro:property name="M_PI" value="3.141592"/>
@@ -48,18 +51,20 @@
   <xacro:macro name="base1">
     <joint name="swivel_J0" type="revolute">
-        <origin xyz="-0.05 0 ${base_height/2 + rplidar_length/2}" rpy="0 0 0" />
+        <origin xyz="-0.05 0 0.15" rpy="0 0 0" />
         <parent link="base_link"/>
         <child link="yaw_Link"/>
         <axis xyz="0 0 1" />
-        <limit lower="-3" upper="3" effort="15.0" velocity="15.0" />
+        <!--<limit lower="-3" upper="3" effort="15.0" velocity="15.0" />-->
+        <limit lower="-0.785" upper="0.785" effort="10.0" velocity="1.0" />
+        <joint_properties damping="0.0" friction="0.0"/>
     </joint>
          <link name="yaw_Link">
-            <inertial>
-                <mass value="0.1" />
+             <!--<inertial>
+                <mass value="4" />
                 <origin xyz="0 0 0" />
-                <inertia ixx="0.01" ixy="0.0" ixz="0.0"
-                         iyy="0.01" iyz="0.0"
-                         izz="0.01" />
-            </inertial>
+                <inertia ixx="4.0" ixy="0.0" ixz="0.0"
+                         iyy="4.0" iyz="0.0"
+                         izz="4.0" />
+            </inertial>-->
             <visual>
                 <origin xyz=" 0 0 0 " rpy="0 0 0" />
@@ -75,9 +80,10 @@
                 </geometry>
             </collision>
+         <cylinder_inertial_matrix  m="1" r="0.025" h="0.2" />
         </link>
-        <gazebo reference=yaw_Link">
+       <!-- <gazebo reference=yaw_Link">
             <material>Gazebo/Black</material>
-        </gazebo>
-    <transmission name="tran1">
+        </gazebo>-->
+   <transmission name="tran1">
     <type>transmission_interface/SimpleTransmission</type>
     <joint name="swivel_J0">
@@ -93,9 +99,9 @@
   <xacro:macro name="base2">
      <joint name="swivel_J1" type="revolute">
-       <origin xyz="-0.02 0 0.16"/>
+       <origin xyz="0.04 0 0.05"/>
        <parent link="yaw_Link"/>
        <child link="pitch_Link"/>
-    <axis xyz="1 0 0" />
-    <limit lower="-0.785" upper="0.785" effort="1.0" velocity="1.0" />
+    <axis xyz="0 1 0" />
+    <limit lower="-0.785" upper="0.785" effort="10.0" velocity="1.0" />
     <joint_properties damping="0.0" friction="0.0"/>
      </joint>
@@ -160,4 +166,12 @@
            </geometry>
       </collision>
+      <surface>
+          <friction>
+            <ode>
+              <mu>0.1</mu>
+              <mu2>0.1</mu2>
+            </ode>
+          </friction>
+        </surface>
       <cylinder_inertial_matrix  m="${wheel_mass}" r="${wheel_radius}" h="${wheel_length}" />
      </link>
@@ -169,8 +183,10 @@
          <type>transmission_interface/SimpleTransmission</type>
          <joint name="${prefix1}_${prefix2}_wheel_joint" >
-             <hardwareInterface>hardware_interface/VelocityJointInterface</hardwareInterface>
+             <!--<hardwareInterface>hardware_interface/VelocityJointInterface</hardwareInterface>-->
+             <hardwareInterface>EffortJointInterface</hardwareInterface>
          </joint>
          <actuator name="${prefix1}_${prefix2}_wheel_joint_motor">
-             <hardwareInterface>hardware_interface/VelocityJointInterface</hardwareInterface>
+             <!--<hardwareInterface>hardware_interface/VelocityJointInterface</hardwareInterface>-->
+             <hardwareInterface>EffortJointInterface</hardwareInterface>
              <mechanicalReduction>1</mechanicalReduction>
          </actuator>
@@ -216,5 +232,6 @@
    <!-- controller -->
 <gazebo>
-  <plugin name="skid_steer_drive_controller" filename="libgazebo_ros_skid_steer_drive.so">
+  <!--<plugin name="skid_steer_drive_controller" filename="libgazebo_ros_skid_steer_drive.so">-->
+  <plugin name="mecanum_controller" filename="libgazebo_ros_planar_move.so">
       <rosDebugLevel>Debug</rosDebugLevel>
        <publishWheelTF>true</publishWheelTF>
@@ -223,5 +240,5 @@
        <alwaysOn>true</alwaysOn>
     <updateRate>100.0</updateRate>
-    <robotNamespace>/</robotNamespace>
+    <robotNamespace>/swivel</robotNamespace>
     <leftFrontJoint>left_front_wheel_joint</leftFrontJoint>
     <rightFrontJoint>right_front_wheel_joint</rightFrontJoint>
@@ -232,5 +249,5 @@
     <broadcastTF>1</broadcastTF>
     <robotBaseFrame>base_footprint</robotBaseFrame>
-    <torque>20</torque>
+    <torque>2</torque>
     <commandTopic>cmd_vel</commandTopic>
     <odometryFrame>odom</odometryFrame>
@@ -378,5 +395,5 @@
 <gazebo>
       <plugin name="gazebo_ros_control" filename="libgazebo_ros_control.so">
-         <robotNamespace>/swivel/swivel</robotNamespace>
+         <robotNamespace>/swivel</robotNamespace>
         <controlPeriod>0.01</controlPeriod>
         <robotSimType>gazebo_ros_control/DefaultRobotHWSim</robotSimType>
